File: hardware/vasvas.kicad_pcb (KiCad board)
At the start: 2 copper layers, 71.1 x 50.8 mm, 31 parts, among them U1 DIP-8_W7.62mm

Commit message: Update vasvas.kicad_pcb
Parts:
- added R11: R_Axial_DIN0207_L6.3mm_D2.5mm_P7.62mm_Horizontal, Resistor_THT:R_Axial_DIN0207_L6.3mm_D2.5mm_P7.62mm_Horizontal, F.Cu at (113.0, 63.5)
- added R12: R_Axial_DIN0207_L6.3mm_D2.5mm_P7.62mm_Horizontal, Resistor_THT:R_Axial_DIN0207_L6.3mm_D2.5mm_P7.62mm_Horizontal, F.Cu at (135.9, 63.5)
Routing:
- net GND: track 217.4 -> 198.3 mm, vias 8 -> 7
- net (no net): track 421.4 -> 425.5 mm
Other:
- board text added: "Stone Voices VasVas base"
- board text removed: "Stone Voices VasVas v1.0"
