File: hardware/vasvas.kicad_sch (KiCad schematic)
At the start: 43 parts, among them J1 Power, J2 Out Left|Stereo, J3 Out Right, J6 Conn 01x20 Socket, J7 Conn 01x20 Socket, SW1 {dblquote}Freeze{dblquote}, U1 NJM4580, Y1 Piezoelement Left, Y2 Piezoelement Right

Commit message: Update vasvas.kicad_sch
Parts:
- U1: value NJM4580 -> 4580DD
- renumbered J6 to J4, J7 to J5
Changed lines of the file:
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@@
 		(on_board yes)
 		(dnp no)
-		(property "Reference" "J7"
+		(property "Reference" "J5"
 			(at 209.042 161.29 0)
 			(effects
@@
 			(project "vasvas"
 				(path "/71d40baf-5761-4982-8ee0-de7cfff85769"
-					(reference "J7")
+					(reference "J5")
 					(unit 1)
 				)
@@
 			)
 		)
-		(property "Value" "NJM4580"
+		(property "Value" "4580DD"
 			(at 72.39 66.04 0)
 			(effects
@@
 		(on_board yes)
 		(dnp no)
-		(property "Reference" "J6"
+		(property "Reference" "J4"
 			(at 142.24 159.258 0)
 			(effects
@@
 			(project "vasvas"
 				(path "/71d40baf-5761-4982-8ee0-de7cfff85769"
-					(reference "J6")
+					(reference "J4")
 					(unit 1)
 				)
@@
 			)
 		)
-		(property "Value" "NJM4580"
+		(property "Value" "4580DD"
 			(at 72.39 31.75 0)
 			(effects

Commit message: Update vasvas.kicad_sch
Connections:
- net GND: now also HL1.1 (K), HL2.1 (K); no longer R11.2, R12.2
- net at R12.1: now also A1.29 (DAC_OUT2), J4.12 (Pin_12); no longer HL2.1 (K)
- net at A1.38 (3V3_D), J4.3 (Pin_3): now also R11.1; no longer HL1.2 (A)
- new net: HL2.2 (A), R12.2
- new net: HL1.2 (A), R11.2
Other:
- moved on the sheet: HL1, HL2, R11, R12
Changed lines of the file:
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@@
 	)
 	(junction
+		(at 97.79 107.95)
+		(diameter 0)
+		(color 0 0 0 0)
+	)
+	(junction
 		(at 97.79 58.42)
 		(diameter 0)
@@
 	)
 	(junction
-		(at 97.79 107.95)
-		(diameter 0)
-		(color 0 0 0 0)
-	)
-	(junction
 		(at 205.74 124.46)
 		(diameter 0)
@@
 	(wire
 		(pts
-			(xy 68.58 107.95) (xy 73.66 107.95)
-		)
-		(stroke
-			(width 0)
-			(type default)
-		)
-	)
-	(wire
-		(pts
 			(xy 205.74 121.92) (xy 214.63 121.92)
 		)
@@
 	(wire
 		(pts
-			(xy 81.28 91.44) (xy 85.09 91.44)
+			(xy 64.77 91.44) (xy 73.66 91.44)
 		)
 		(stroke
@@
 	(wire
 		(pts
-			(xy 97.79 107.95) (xy 97.79 111.76)
+			(xy 97.79 91.44) (xy 97.79 107.95)
 		)
 		(stroke
@@
 	(wire
 		(pts
-			(xy 92.71 107.95) (xy 97.79 107.95)
+			(xy 137.16 132.08) (xy 142.24 132.08)
 		)
 		(stroke
@@
 	(wire
 		(pts
-			(xy 137.16 132.08) (xy 142.24 132.08)
+			(xy 29.21 173.99) (xy 55.88 173.99)
 		)
 		(stroke
@@
 	(wire
 		(pts
-			(xy 29.21 173.99) (xy 55.88 173.99)
+			(xy 128.27 132.08) (xy 137.16 132.08)
 		)
 		(stroke
@@
 	(wire
 		(pts
-			(xy 128.27 132.08) (xy 137.16 132.08)
+			(xy 81.28 107.95) (xy 85.09 107.95)
 		)
 		(stroke
@@
 	(wire
 		(pts
-			(xy 97.79 91.44) (xy 97.79 107.95)
-		)
-		(stroke
-			(width 0)
-			(type default)
-		)
-	)
-	(wire
-		(pts
 			(xy 257.81 59.69) (xy 257.81 63.5)
 		)
@@
 	(wire
 		(pts
+			(xy 92.71 107.95) (xy 97.79 107.95)
+		)
+		(stroke
+			(width 0)
+			(type default)
+		)
+	)
+	(wire
+		(pts
 			(xy 137.16 127) (xy 142.24 127)
 		)
@@
 	(wire
 		(pts
-			(xy 128.27 129.54) (xy 137.16 129.54)
+			(xy 68.58 107.95) (xy 73.66 107.95)
 		)
 		(stroke
@@
 	(wire
 		(pts
-			(xy 245.11 52.07) (xy 260.35 52.07)
+			(xy 128.27 129.54) (xy 137.16 129.54)
 		)
 		(stroke
@@
 	(wire
 		(pts
-			(xy 81.28 107.95) (xy 85.09 107.95)
+			(xy 245.11 52.07) (xy 260.35 52.07)
 		)
 		(stroke
@@
 	(wire
 		(pts
-			(xy 92.71 91.44) (xy 97.79 91.44)
-		)
-		(stroke
-			(width 0)
-			(type default)
-		)
-	)
-	(wire
-		(pts
-			(xy 64.77 91.44) (xy 73.66 91.44)
+			(xy 214.63 101.6) (xy 205.74 101.6)
 		)
 		(stroke
@@
 	(wire
 		(pts
-			(xy 214.63 101.6) (xy 205.74 101.6)
+			(xy 137.16 149.86) (xy 142.24 149.86)
 		)
 		(stroke
@@
 	(wire
 		(pts
-			(xy 137.16 149.86) (xy 142.24 149.86)
+			(xy 260.35 30.48) (xy 254 30.48)
 		)
 		(stroke
@@
 	(wire
 		(pts
-			(xy 260.35 30.48) (xy 254 30.48)
+			(xy 45.72 82.55) (xy 45.72 127)
 		)
 		(stroke
@@
 	(wire
 		(pts
-			(xy 45.72 82.55) (xy 45.72 127)
+			(xy 80.01 58.42) (xy 80.01 73.66)
 		)
 		(stroke
@@
 	(wire
 		(pts
-			(xy 80.01 58.42) (xy 80.01 73.66)
+			(xy 200.66 132.08) (xy 205.74 132.08)
 		)
 		(stroke
@@
 	(wire
 		(pts
-			(xy 200.66 132.08) (xy 205.74 132.08)
+			(xy 92.71 91.44) (xy 97.79 91.44)
 		)
 		(stroke
@@
 	(wire
 		(pts
+			(xy 81.28 91.44) (xy 85.09 91.44)
+		)
+		(stroke
+			(width 0)
+			(type default)
+		)
+	)
+	(wire
+		(pts
 			(xy 134.62 69.85) (xy 149.86 69.85)
 		)
@@
 	(wire
 		(pts
+			(xy 97.79 107.95) (xy 97.79 111.76)
+		)
+		(stroke
+			(width 0)
+			(type default)
+		)
+	)
+	(wire
+		(pts
 			(xy 205.74 149.86) (xy 214.63 149.86)
 		)
@@
 	(symbol
 		(lib_id "Device:R")
-		(at 88.9 107.95 90)
+		(at 77.47 107.95 90)
 		(unit 1)
 		(exclude_from_sim no)
@@
 		(fields_autoplaced yes)
 		(property "Reference" "R12"
-			(at 88.9 101.6 90)
+			(at 77.47 101.6 90)
 			(effects
 				(font
@@
 		)
 		(property "Value" "510"
-			(at 88.9 104.14 90)
+			(at 77.47 104.14 90)
 			(effects
 				(font
@@
 		)
 		(property "Footprint" "Resistor_SMD:R_0805_2012Metric"
-			(at 88.9 109.728 90)
+			(at 77.47 109.728 90)
 			(effects
 				(font
@@
 		)
 		(property "Datasheet" "~"
-			(at 88.9 107.95 0)
+			(at 77.47 107.95 0)
 			(effects
 				(font
@@
 		)
 		(property "Description" ""
-			(at 88.9 107.95 0)
+			(at 77.47 107.95 0)
 			(effects
 				(font
@@
 	(symbol
 		(lib_id "Device:LED")
-		(at 77.47 107.95 180)
+		(at 88.9 107.95 180)
 		(unit 1)
 		(exclude_from_sim no)
@@
 		(dnp no)
 		(property "Reference" "HL2"
-			(at 79.0575 114.3 0)
+			(at 90.4875 114.3 0)
 			(effects
 				(font
@@
 		)
 		(property "Value" "{dblquote}Freeze{dblquote}"
-			(at 79.0575 111.76 0)
+			(at 90.4875 111.76 0)
 			(effects
 				(font
@@
 		)
 		(property "Footprint" ""
-			(at 77.47 107.95 0)
+			(at 88.9 107.95 0)
 			(effects
 				(font
@@
 		)
 		(property "Datasheet" "~"
-			(at 77.47 107.95 0)
+			(at 88.9 107.95 0)
 			(effects
 				(font
@@
 		)
 		(property "Description" "Light emitting diode"
-			(at 77.47 107.95 0)
+			(at 88.9 107.95 0)
 			(effects
 				(font
@@
 		)
 		(property "Sim.Pins" "1=K 2=A"
-			(at 77.47 107.95 0)
+			(at 88.9 107.95 0)
 			(effects
 				(font
@@
 	(symbol
 		(lib_id "Device:LED")
-		(at 77.47 91.44 180)
+		(at 88.9 91.44 180)
 		(unit 1)
 		(exclude_from_sim no)
@@
 		(dnp no)
 		(property "Reference" "HL1"
-			(at 79.0575 97.79 0)
+			(at 90.4875 97.79 0)
 			(effects
 				(font
@@
 		)
 		(property "Value" "{dblquote}Power{dblquote}"
-			(at 79.0575 95.25 0)
+			(at 90.4875 95.25 0)
 			(effects
 				(font
@@
 		)
 		(property "Footprint" ""
-			(at 77.47 91.44 0)
+			(at 88.9 91.44 0)
 			(effects
 				(font
@@
 		)
 		(property "Datasheet" "~"
-			(at 77.47 91.44 0)
+			(at 88.9 91.44 0)
 			(effects
 				(font
@@
 		)
 		(property "Description" "Light emitting diode"
-			(at 77.47 91.44 0)
+			(at 88.9 91.44 0)
 			(effects
 				(font
@@
 		)
 		(property "Sim.Pins" "1=K 2=A"
-			(at 77.47 91.44 0)
+			(at 88.9 91.44 0)
 			(effects
 				(font
@@
 	(symbol
 		(lib_id "Device:R")
-		(at 88.9 91.44 90)
+		(at 77.47 91.44 90)
 		(unit 1)
 		(exclude_from_sim no)
@@
 		(fields_autoplaced yes)
 		(property "Reference" "R11"
-			(at 88.9 85.09 90)
+			(at 77.47 85.09 90)
 			(effects
 				(font
@@
 		)
 		(property "Value" "510"
-			(at 88.9 87.63 90)
+			(at 77.47 87.63 90)
 			(effects
 				(font
@@
 		)
 		(property "Footprint" "Resistor_SMD:R_0805_2012Metric"
-			(at 88.9 93.218 90)
+			(at 77.47 93.218 90)
 			(effects
 				(font
@@
 		)
 		(property "Datasheet" "~"
-			(at 88.9 91.44 0)
+			(at 77.47 91.44 0)
 			(effects
 				(font
@@
 		)
 		(property "Description" ""
-			(at 88.9 91.44 0)
+			(at 77.47 91.44 0)
 			(effects
 				(font
